Commit message: add planner

File: src/simplebot_description/urdf/simplebot.xacro (robot description, xacro)
@@ -110,5 +110,5 @@
   <parent link="base_link"/>
   <child link="right_wheel_1"/>
-  <axis xyz="0.0 -1.0 0.0"/>
+  <axis xyz="0.0 1.0 0.0"/>
 </joint>
 <joint name="Rev2" type="continuous">

File: src/steer_wheel_bot/steer_wheel_bot_description/urdf/mobile_mover.xacro (robot description, xacro)
@@ -288,5 +288,5 @@
   <parent link="base_link"/>
   <child link="front_right_steer_1"/>
-  <axis xyz="-0.0 0.0 1.0"/>
+  <axis xyz="0.0 0.0 1.0"/>
   <limit effort="100" lower="-0.923599" upper="0.923599" velocity="100"/>
 </joint>
@@ -295,5 +295,5 @@
   <parent link="base_link"/>
   <child link="front_left_steer_1"/>
-  <axis xyz="-0.0 0.0 1.0"/>
+  <axis xyz="0.0 0.0 1.0"/>
   <limit effort="100" lower="-0.923599" upper="0.923599" velocity="100"/>
 </joint>
@@ -322,5 +322,5 @@
   <parent link="base_link"/>
   <child link="front_steer_1"/>
-  <axis xyz="0.0 -0.0 1.0"/>
+  <axis xyz="0.0 0.0 1.0"/>
 </joint>
 <joint name="front_right_wheel_joint" type="continuous">
@@ -328,5 +328,5 @@
   <parent link="front_right_steer_1"/>
   <child link="front_right_wheel_1"/>
-   <axis xyz="-0.038364 0.999264 0.0"/>
+   <axis xyz="0.0 1.0 0.0"/>
 </joint>
 <joint name="front_left_wheel_joint" type="continuous">
@@ -334,5 +334,5 @@
   <parent link="front_left_steer_1"/>
   <child link="front_left_wheel_1"/>
-   <axis xyz="-0.038364 0.999264 0.0"/>
+   <axis xyz="0.0 1.0 0.0"/>
 </joint>
 <joint name="Rigid66" type="fixed">
@@ -351,5 +351,5 @@
   <parent link="base_link"/>
   <child link="rear_left_wheel_1"/>
-  <axis xyz="-0.0 1.0 -0.0"/>
+  <axis xyz="0.0 1.0 0.0"/>
 </joint>
 <joint name="rear_right_wheel_joint" type="continuous">
@@ -357,5 +357,5 @@
   <parent link="base_link"/>
   <child link="rear_right_wheel_1"/>
-  <axis xyz="-0.0 1.0 -0.0"/>
+  <axis xyz="0.0 1.0 0.0"/>
 </joint>
 </robot>
